Commit message: transform sync boilerplate integration

File: sting3dengine/assets/urdf/plane.urdf (robot description, URDF)
Before this commit: robot plane, 1 links, 0 joints
Links:
- link planeLink: mass 0 -> .0; geometry collision box size=30 10 30

Commit message: made ground plane wide enough to accomodate more floor space

File: sting3dengine/assets/urdf/plane.urdf (robot description, URDF)
Before this commit: robot plane, 1 links, 0 joints
Links:
- link planeLink: geometry collision box size=3000 10 3000
